File: KiCad9_Data/miniFanForSoldering.kicad_sch (KiCad schematic)
At the start: 28 parts, among them J1 Conn_01x02_Socket, J2 Conn_01x02_Pin, M1 5V 0.3A, Q1 2SC4811, SW1 SW_SPDT, SW2 SW_SPDT, U2 L7805, U4 L7805

Commit message: libフォルダを追加した。また回路図のシンボルもそれに合わせて書き直した（ライブラリ２つを登録してください）
Parts:
- removed U1: ~, symbol New_Library:HC-SR04
- added U1: ~, symbol New_Lib:HC-SR04
Connections:
- net GND: now also U1.4 (GND)
- net at A1.39 (VSYS), C3.1, C4.1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: now also U1.1 (Vcc)
- net at A1.5 (GPIO3): now also U1.2 (Trig)
- net at R1.1: now also U1.3 (Echo)
